File: projetoFinal.kicad_sch (KiCad schematic)
At the start: 31 parts

Commit message: coloquei uns footprint e deve estar tudo errado
Parts:
- C1, C9: value (none) -> 4700uF; footprint (none) -> Capacitor_THT:CP_Radial_Tantal_D6.0mm_P5.00mm
- C10, C2, C4, C8: value (none) -> 100nF; footprint (none) -> Capacitor_THT:C_Axial_L3.8mm_D2.6mm_P7.50mm_Horizontal
- C3, C7: value (none) -> 100uF; footprint (none) -> Capacitor_THT:C_Axial_L3.8mm_D2.6mm_P7.50mm_Horizontal
- C5, C6: value (none) -> 10uF; footprint (none) -> Capacitor_THT:C_Axial_L3.8mm_D2.6mm_P7.50mm_Horizontal
- D1, D2, D5: value (none) -> 1N4004; footprint (none) -> Diode_THT:D_A-405_P10.16mm_Horizontal
- D3: value (none) -> GBU4A; footprint (none) -> Diode_THT:Diode_Bridge_Vishay_GBU
- D4: renamed from D5; value (none) -> 1N4004; footprint (none) -> Diode_THT:D_A-405_P10.16mm_Horizontal
- D6: footprint (none) -> Diode_THT:D_A-405_P10.16mm_Horizontal
- HS1: renamed from HS?; value (none) -> Heatsink; footprint (none) -> xHeatsink:Heatsink_AAVID_573300D00010G_TO-263
- HS2: renamed from HS?; footprint (none) -> xHeatsink:Heatsink_AAVID_573300D00010G_TO-263
- J1, J3, J4, J5: value (none) -> Conn_01x01_Male; footprint (none) -> MountingHole:MountingHole_2.2mm_M2_DIN965_Pad
- J2, J6: value (none) -> Conn_01x04
- R1, R2: value (none) -> 240; footprint (none) -> Resistor_THT:R_Axial_DIN0204_L3.6mm_D1.6mm_P7.62mm_Horizontal
- R3: value (none) -> 1k; footprint (none) -> Resistor_THT:R_Axial_DIN0204_L3.6mm_D1.6mm_P7.62mm_Horizontal
- RV1, RV2: value (none) -> R_Potentiometer; footprint (none) -> Potentiometer_THT:Potentiometer_Piher_T-16L_Single_Vertical_Hole
- U1: value (none) -> LM317_TO-220; footprint (none) -> Package_TO_SOT_THT:TO-220-3_Vertical
- U2: value (none) -> LM337_TO220; footprint (none) -> Package_TO_SOT_THT:TO-220-3_Vertical
