File: _autosave-projetoFinal.kicad_sch (KiCad schematic)
At the start: 31 parts, among them J1 Conn_01x01_Male, J2 Conn_01x04, J3 Conn_01x01_Male, J4 Conn_01x01_Male, J5 Conn_01x01_Male, J6 Conn_01x04, U1 LM317_TO-220, U2 LM337_TO220

Commit message: footprints quase certos
Parts:
- C10, C2, C4, C8: footprint Capacitor_THT:C_Axial_L3.8mm_D2.6mm_P7.50mm_Horizontal -> Capacitor_THT:C_Disc_D3.0mm_W2.0mm_P2.50mm
- C3, C7: footprint Capacitor_THT:C_Axial_L3.8mm_D2.6mm_P7.50mm_Horizontal -> Capacitor_THT:CP_Radial_D7.5mm_P2.50mm
- C5, C6: footprint Capacitor_THT:C_Axial_L3.8mm_D2.6mm_P7.50mm_Horizontal -> Capacitor_THT:CP_Radial_D5.0mm_P2.50mm
- J1, J3, J4, J5: footprint MountingHole:MountingHole_2.2mm_M2_DIN965_Pad -> footprints:Banana_Jack_1Pin
Changed lines of the file:
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@@
       (effects (font (size 1.27 1.27)) (justify left))
     )
-    (property "Footprint" "Capacitor_THT:C_Axial_L3.8mm_D2.6mm_P7.50mm_Horizontal" (id 2) (at 186.3852 111.76 0)
+    (property "Footprint" "Capacitor_THT:CP_Radial_D7.5mm_P2.50mm" (id 2) (at 186.3852 111.76 0)
       (effects (font (size 1.27 1.27)) hide)
     )
@@
       (effects (font (size 1.27 1.27)) (justify left))
     )
-    (property "Footprint" "Capacitor_THT:C_Axial_L3.8mm_D2.6mm_P7.50mm_Horizontal" (id 2) (at 166.0652 107.95 0)
+    (property "Footprint" "Capacitor_THT:CP_Radial_D5.0mm_P2.50mm" (id 2) (at 166.0652 107.95 0)
       (effects (font (size 1.27 1.27)) hide)
     )
@@
       (effects (font (size 1.27 1.27)) (justify left))
     )
-    (property "Footprint" "Capacitor_THT:C_Axial_L3.8mm_D2.6mm_P7.50mm_Horizontal" (id 2) (at 136.8552 88.9 0)
+    (property "Footprint" "Capacitor_THT:C_Disc_D3.0mm_W2.0mm_P2.50mm" (id 2) (at 136.8552 88.9 0)
       (effects (font (size 1.27 1.27)) hide)
     )
@@
       (effects (font (size 1.27 1.27)) hide)
     )
-    (property "Footprint" "MountingHole:MountingHole_2.2mm_M2_DIN965_Pad" (id 2) (at 220.98 102.87 0)
+    (property "Footprint" "footprints:Banana_Jack_1Pin" (id 2) (at 220.98 102.87 0)
       (effects (font (size 1.27 1.27)) hide)
     )
@@
       (effects (font (size 1.27 1.27)) hide)
     )
-    (property "Footprint" "MountingHole:MountingHole_2.2mm_M2_DIN965_Pad" (id 2) (at 220.98 124.46 0)
+    (property "Footprint" "footprints:Banana_Jack_1Pin" (id 2) (at 220.98 124.46 0)
       (effects (font (size 1.27 1.27)) hide)
     )
@@
       (effects (font (size 1.27 1.27)) hide)
     )
-    (property "Footprint" "MountingHole:MountingHole_2.2mm_M2_DIN965_Pad" (id 2) (at 220.98 90.17 0)
+    (property "Footprint" "footprints:Banana_Jack_1Pin" (id 2) (at 220.98 90.17 0)
       (effects (font (size 1.27 1.27)) hide)
     )
@@
       (effects (font (size 1.27 1.27)) (justify left))
     )
-    (property "Footprint" "Capacitor_THT:C_Axial_L3.8mm_D2.6mm_P7.50mm_Horizontal" (id 2) (at 206.7052 93.98 0)
+    (property "Footprint" "Capacitor_THT:C_Disc_D3.0mm_W2.0mm_P2.50mm" (id 2) (at 206.7052 93.98 0)
       (effects (font (size 1.27 1.27)) hide)
     )
@@
       (effects (font (size 1.27 1.27)) hide)
     )
-    (property "Footprint" "MountingHole:MountingHole_2.2mm_M2_DIN965_Pad" (id 2) (at 220.98 71.12 0)
+    (property "Footprint" "footprints:Banana_Jack_1Pin" (id 2) (at 220.98 71.12 0)
       (effects (font (size 1.27 1.27)) hide)
     )
@@
       (effects (font (size 1.27 1.27)) (justify left))
     )
-    (property "Footprint" "Capacitor_THT:C_Axial_L3.8mm_D2.6mm_P7.50mm_Horizontal" (id 2) (at 186.3852 88.9 0)
+    (property "Footprint" "Capacitor_THT:CP_Radial_D7.5mm_P2.50mm" (id 2) (at 186.3852 88.9 0)
       (effects (font (size 1.27 1.27)) hide)
     )
@@
       (effects (font (size 1.27 1.27)) (justify left))
     )
-    (property "Footprint" "Capacitor_THT:C_Axial_L3.8mm_D2.6mm_P7.50mm_Horizontal" (id 2) (at 166.0652 95.25 0)
+    (property "Footprint" "Capacitor_THT:CP_Radial_D5.0mm_P2.50mm" (id 2) (at 166.0652 95.25 0)
       (effects (font (size 1.27 1.27)) hide)
     )
@@
       (effects (font (size 1.27 1.27)) (justify left))
     )
-    (property "Footprint" "Capacitor_THT:C_Axial_L3.8mm_D2.6mm_P7.50mm_Horizontal" (id 2) (at 136.8552 111.76 0)
+    (property "Footprint" "Capacitor_THT:C_Disc_D3.0mm_W2.0mm_P2.50mm" (id 2) (at 136.8552 111.76 0)
       (effects (font (size 1.27 1.27)) hide)
     )
@@
       (effects (font (size 1.27 1.27)) (justify left))
     )
-    (property "Footprint" "Capacitor_THT:C_Axial_L3.8mm_D2.6mm_P7.50mm_Horizontal" (id 2) (at 206.7052 106.68 0)
+    (property "Footprint" "Capacitor_THT:C_Disc_D3.0mm_W2.0mm_P2.50mm" (id 2) (at 206.7052 106.68 0)
       (effects (font (size 1.27 1.27)) hide)
     )
@@
     )
     (path "/1ade4dff-4c0c-4a8d-a0a5-4714a29520b8"
-      (reference "C2") (unit 1) (value "100nF") (footprint "Capacitor_THT:C_Axial_L3.8mm_D2.6mm_P7.50mm_Horizontal")
+      (reference "C2") (unit 1) (value "100nF") (footprint "Capacitor_THT:C_Disc_D3.0mm_W2.0mm_P2.50mm")
     )
     (path "/41f3443a-b913-4576-be7a-ee23ccd054d8"
-      (reference "C3") (unit 1) (value "100uF") (footprint "Capacitor_THT:C_Axial_L3.8mm_D2.6mm_P7.50mm_Horizontal")
+      (reference "C3") (unit 1) (value "100uF") (footprint "Capacitor_THT:CP_Radial_D7.5mm_P2.50mm")
     )
     (path "/41c365fa-3d50-4050-8aef-1622d6a45dc7"
-      (reference "C4") (unit 1) (value "100nF") (footprint "Capacitor_THT:C_Axial_L3.8mm_D2.6mm_P7.50mm_Horizontal")
+      (reference "C4") (unit 1) (value "100nF") (footprint "Capacitor_THT:C_Disc_D3.0mm_W2.0mm_P2.50mm")
     )
     (path "/425a6059-a32f-470e-8724-52feef15c5a2"
-      (reference "C5") (unit 1) (value "10uF") (footprint "Capacitor_THT:C_Axial_L3.8mm_D2.6mm_P7.50mm_Horizontal")
+      (reference "C5") (unit 1) (value "10uF") (footprint "Capacitor_THT:CP_Radial_D5.0mm_P2.50mm")
     )
     (path "/0a97405b-8e34-4959-aa6c-34385c8a16b7"
-      (reference "C6") (unit 1) (value "10uF") (footprint "Capacitor_THT:C_Axial_L3.8mm_D2.6mm_P7.50mm_Horizontal")
+      (reference "C6") (unit 1) (value "10uF") (footprint "Capacitor_THT:CP_Radial_D5.0mm_P2.50mm")
     )
     (path "/09ca0643-81ba-4cf0-9ba1-a08513b96e39"
-      (reference "C7") (unit 1) (value "100uF") (footprint "Capacitor_THT:C_Axial_L3.8mm_D2.6mm_P7.50mm_Horizontal")
+      (reference "C7") (unit 1) (value "100uF") (footprint "Capacitor_THT:CP_Radial_D7.5mm_P2.50mm")
     )
     (path "/cd752140-16af-492a-820f-0d702db332c5"
-      (reference "C8") (unit 1) (value "100nF") (footprint "Capacitor_THT:C_Axial_L3.8mm_D2.6mm_P7.50mm_Horizontal")
+      (reference "C8") (unit 1) (value "100nF") (footprint "Capacitor_THT:C_Disc_D3.0mm_W2.0mm_P2.50mm")
     )
     (path "/84bd8a6e-265c-493e-a929-a6e637651e39"
@@
     )
     (path "/a6344f07-d3bf-43c5-bc47-4d2fb281ba23"
-      (reference "C10") (unit 1) (value "100nF") (footprint "Capacitor_THT:C_Axial_L3.8mm_D2.6mm_P7.50mm_Horizontal")
+      (reference "C10") (unit 1) (value "100nF") (footprint "Capacitor_THT:C_Disc_D3.0mm_W2.0mm_P2.50mm")
     )
     (path "/d737ca12-6267-4de2-992c-2c978c7454e2"
@@
     )
     (path "/41cb776f-97db-4442-99b7-259c4cf7a394"
-      (reference "J1") (unit 1) (value "Conn_01x01_Male") (footprint "MountingHole:MountingHole_2.2mm_M2_DIN965_Pad")
+      (reference "J1") (unit 1) (value "Conn_01x01_Male") (footprint "footprints:Banana_Jack_1Pin")
     )
     (path "/89c7a74c-1139-4479-9e68-735b14ceb39f"
@@
     )
     (path "/37f109e5-454c-4bf7-b002-0195ee51cad8"
-      (reference "J3") (unit 1) (value "Conn_01x01_Male") (footprint "MountingHole:MountingHole_2.2mm_M2_DIN965_Pad")
+      (reference "J3") (unit 1) (value "Conn_01x01_Male") (footprint "footprints:Banana_Jack_1Pin")
     )
     (path "/2e338e8c-2371-44aa-8260-c10d66f52735"
-      (reference "J4") (unit 1) (value "Conn_01x01_Male") (footprint "MountingHole:MountingHole_2.2mm_M2_DIN965_Pad")
+      (reference "J4") (unit 1) (value "Conn_01x01_Male") (footprint "footprints:Banana_Jack_1Pin")
     )
     (path "/30e41159-5267-46e6-8d9c-1174e7b44836"
-      (reference "J5") (unit 1) (value "Conn_01x01_Male") (footprint "MountingHole:MountingHole_2.2mm_M2_DIN965_Pad")
+      (reference "J5") (unit 1) (value "Conn_01x01_Male") (footprint "footprints:Banana_Jack_1Pin")
     )
     (path "/57f31529-1499-458f-9a48-eb59bb575b06"
