File: _autosave-projetoFinal.kicad_pcb (KiCad board)
At the start: 2 copper layers, 30 parts, among them J1 Conn_01x01_Male, J2 Conn_01x04, J3 Conn_01x01_Male, J4 Conn_01x01_Male, J5 Conn_01x01_Male, J6 Conn_01x04, U1 LM317_TO-220, U2 LM337_TO220

Commit message: roteamento feito
Parts:
- added HS1: Heatsink, Heatsink:Heatsink_Stonecold_HS-132_32x14mm_2xFixation1.5mm, F.Cu at (104.1, 158.4)
- added J7: Conn_01x02, TerminalBlock_Phoenix:TerminalBlock_Phoenix_MKDS-1,5-2_1x02_P5.00mm_Horizontal, F.Cu at (60.7, 105.5)
- C1, C9: footprint Capacitor_THT:CP_Radial_Tantal_D6.0mm_P5.00mm -> Capacitor_THT:CP_Radial_D10.0mm_P2.50mm
- C10, C2, C4, C8: footprint Capacitor_THT:C_Axial_L3.8mm_D2.6mm_P7.50mm_Horizontal -> Capacitor_THT:C_Disc_D3.0mm_W2.0mm_P2.50mm
- C3, C7: footprint Capacitor_THT:C_Axial_L3.8mm_D2.6mm_P7.50mm_Horizontal -> Capacitor_THT:CP_Radial_D7.5mm_P2.50mm
- C5, C6: footprint Capacitor_THT:C_Axial_L3.8mm_D2.6mm_P7.50mm_Horizontal -> Capacitor_THT:CP_Radial_D5.0mm_P2.50mm
- D1, D2, D4, D5: footprint Diode_THT:D_A-405_P10.16mm_Horizontal -> Diode_THT:D_5W_P10.16mm_Horizontal
- D6: footprint Diode_THT:D_A-405_P10.16mm_Horizontal -> LED_THT:LED_D5.0mm
- J1, J3, J4, J5: footprint MountingHole:MountingHole_2.2mm_M2_DIN965_Pad -> footprints:Banana_Jack_1Pin
- J2: value Conn_01x04 -> Conn_01x02; footprint Connector:FanPinHeader_1x04_P2.54mm_Vertical -> TerminalBlock_Phoenix:TerminalBlock_Phoenix_MKDS-1,5-2_1x02_P5.00mm_Horizontal
- J6: footprint Connector:FanPinHeader_1x04_P2.54mm_Vertical -> Connector_PinHeader_2.54mm:PinHeader_1x04_P2.54mm_Vertical
- R1, R2: footprint Resistor_THT:R_Axial_DIN0204_L3.6mm_D1.6mm_P7.62mm_Horizontal -> Resistor_THT:R_Axial_DIN0207_L6.3mm_D2.5mm_P10.16mm_Horizontal
- moved J2 170.6 mm to (60.7, 94.0), turned to -90 degrees
- moved D6 132.3 mm to (62.2, 142.2), turned to 90 degrees
- moved J6 109.5 mm to (149.9, 132.1), turned to -90 degrees
- moved D1 105.2 mm to (99.1, 141.0)
- moved HS2 99.5 mm to (104.1, 52.0)
- moved U2 99.1 mm to (101.6, 52.9)
- moved C1 90.1 mm to (78.7, 127.0), turned to -90 degrees
- moved R3 88.9 mm to (62.9, 126.4), turned to -90 degrees
- moved RV1 85.1 mm to (99.1, 112.2), turned to -90 degrees
- moved J1 83.6 mm to (165.1, 139.1)
- moved D2 83.4 mm to (129.5, 127.0), turned to -90 degrees
- moved C9 80.2 mm to (74.9, 71.1), turned to -90 degrees
- moved C10 77.2 mm to (85.1, 71.2), turned to -90 degrees
- moved C2 76.4 mm to (88.9, 127.0), turned to -90 degrees
- moved U1 72.3 mm to (106.7, 157.5), turned to 180 degrees
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Connections:
- J2 pad 1: Net-(D3-Pad2) -> GND
- J2 pad 2: GND -> Net-(D3-Pad2)
Routing:
- net GND: track 0.00 -> 305.9 mm
- net Net-(C3-Pad1): track 0.00 -> 110.0 mm
- net Net-(C7-Pad2): track 0.00 -> 99.7 mm
- net Net-(D4-Pad1): track 0.00 -> 88.2 mm
- net Net-(C5-Pad1): track 0.00 -> 69.5 mm
- net Net-(C1-Pad1): track 0.00 -> 66.2 mm
- net Net-(C10-Pad2): track 0.00 -> 46.3 mm
- net Net-(D6-Pad2): track 0.00 -> 5.98 mm
- added copper zone on B.Cu, net (none)
Other:
- board text added: "cu"
